Commit message: updated

File: description/robot_core.xacro (robot description, xacro)
@@ -58,5 +58,5 @@
     </gazebo>
     <!-- LEFT FRONT WHEEL -->
-    <joint name="left_front_wheel_joint" type="continuous">
+    <joint name="left_front_wheel_joint" type="fixed">
         <parent link="base_link"/>
         <child link="left_front_wheel"/>
@@ -71,9 +71,9 @@
             <material name="black"/>
         </visual>
-        <collision>
+        <!--<collision>
             <geometry>
                 <sphere radius="0.0225" />
             </geometry>
-        </collision>
+        </collision> -->
         <xacro:inertial_cylinder mass="0.1" length="0.018" radius="0.0225">
             <origin xyz="0 0 0" rpy="0 0 0"/>
@@ -114,5 +114,5 @@
     </gazebo>
     <!-- RIGHT FRONT WHEEL -->
-    <joint name="right_front_wheel_joint" type="continuous">
+    <joint name="right_front_wheel_joint" type="fixed">
         <parent link="base_link"/>
         <child link="right_front_wheel"/>
@@ -127,9 +127,9 @@
             <material name="black"/>
         </visual>
-        <collision>
+        <!--<collision>
             <geometry>
                 <sphere radius="0.0225" />
             </geometry>
-        </collision>
+        </collision>-->
         <xacro:inertial_cylinder mass="0.1" length="0.018" radius="0.0225">
             <origin xyz="0 0 0" rpy="0 0 0"/>

File: description/ros2_control.xacro (robot description, xacro)
@@ -5,6 +5,6 @@
             <hardware>
                 <plugin>diffdrive_arduino/DiffDriveArduino</plugin>
-                <param name="left_wheel_name">left_wheel_joint</param>
-                <param name="right_wheel_name">right_wheel_joint</param>
+                <param name="left_wheel_name">left_rear_wheel_joint</param>
+                <param name="right_wheel_name">right_rear_wheel_joint</param>
                 <param name="loop_rate">30</param>
                 <param name="device">/dev/ttyACM0</param>
@@ -13,5 +13,13 @@
                 <param name="enc_counts_per_rev">3450</param>
             </hardware>
-            <joint name="left_wheel_joint">
+            <!-- <joint name="left_front_wheel_joint">
+                <command_interface name="velocity">
+                    <param name="min">-10</param>
+                    <param name="max">10</param>
+                </command_interface>
+                <state_interface name="velocity"/>
+                <state_interface name="position"/>
+            </joint> -->
+            <joint name="left_rear_wheel_joint">
                 <command_interface name="velocity">
                     <param name="min">-10</param>
@@ -21,5 +29,5 @@
                 <state_interface name="position"/>
             </joint>
-            <!--<joint name="left_rear_wheel_joint">
+            <!-- <joint name="right_front_wheel_joint">
                 <command_interface name="velocity">
                     <param name="min">-10</param>
@@ -29,5 +37,5 @@
                 <state_interface name="position"/>
             </joint> -->
-            <joint name="right_wheel_joint">
+            <joint name="right_rear_wheel_joint">
                 <command_interface name="velocity">
                     <param name="min">-10</param>
@@ -37,12 +45,4 @@
                 <state_interface name="position"/>
             </joint>
-            <!--<joint name="right_rear_wheel_joint">
-                <command_interface name="velocity">
-                    <param name="min">-10</param>
-                    <param name="max">10</param>
-                </command_interface>
-                <state_interface name="velocity"/>
-                <state_interface name="position"/>
-            </joint> -->
         </ros2_control>
     </xacro:unless>
