Commit message: ros2_control update

File: description/ros2_control.xacro (robot description, xacro)
@@ -11,5 +11,5 @@
                 <param name="baud_rate">57600</param>
                 <param name="timeout">1000</param>
-                <param name="enc_counts_per_rev">500</param>
+                <param name="enc_counts_per_rev">3450</param>
             </hardware>
             <joint name="left_wheel_joint">
@@ -21,5 +21,5 @@
                 <state_interface name="position"/>
             </joint>
-            <joint name="left_rear_wheel_joint">
+            <!--<joint name="left_rear_wheel_joint">
                 <command_interface name="velocity">
                     <param name="min">-10</param>
@@ -28,5 +28,5 @@
                 <state_interface name="velocity"/>
                 <state_interface name="position"/>
-            </joint>
+            </joint> -->
             <joint name="right_wheel_joint">
                 <command_interface name="velocity">
@@ -37,5 +37,5 @@
                 <state_interface name="position"/>
             </joint>
-            <joint name="right_rear_wheel_joint">
+            <!--<joint name="right_rear_wheel_joint">
                 <command_interface name="velocity">
                     <param name="min">-10</param>
@@ -44,5 +44,5 @@
                 <state_interface name="velocity"/>
                 <state_interface name="position"/>
-            </joint>
+            </joint> -->
         </ros2_control>
     </xacro:unless>

Commit message: updated

File: description/ros2_control.xacro (robot description, xacro)
@@ -5,13 +5,13 @@
             <hardware>
                 <plugin>diffdrive_arduino/DiffDriveArduino</plugin>
-                <param name="left_wheel_name">left_wheel_joint</param>
-                <param name="right_wheel_name">right_wheel_joint</param>
+                <param name="left_wheel_name">left_rear_wheel_joint</param>
+                <param name="right_wheel_name">right_rear_wheel_joint</param>
                 <param name="loop_rate">30</param>
                 <param name="device">/dev/ttyACM0</param>
                 <param name="baud_rate">57600</param>
                 <param name="timeout">1000</param>
-                <param name="enc_counts_per_rev">500</param>
+                <param name="enc_counts_per_rev">3450</param>
             </hardware>
-            <joint name="left_wheel_joint">
+            <!-- <joint name="left_front_wheel_joint">
                 <command_interface name="velocity">
                     <param name="min">-10</param>
@@ -20,5 +20,5 @@
                 <state_interface name="velocity"/>
                 <state_interface name="position"/>
-            </joint>
+            </joint> -->
             <joint name="left_rear_wheel_joint">
                 <command_interface name="velocity">
@@ -29,5 +29,5 @@
                 <state_interface name="position"/>
             </joint>
-            <joint name="right_wheel_joint">
+            <!-- <joint name="right_front_wheel_joint">
                 <command_interface name="velocity">
                     <param name="min">-10</param>
@@ -36,5 +36,5 @@
                 <state_interface name="velocity"/>
                 <state_interface name="position"/>
-            </joint>
+            </joint> -->
             <joint name="right_rear_wheel_joint">
                 <command_interface name="velocity">
@@ -88,5 +88,5 @@
     <gazebo>
         <plugin name="gazebo_ros2_control" filename="libgazebo_ros2_control.so">
-            <parameters>$(find )/config/my_controllers.yaml</parameters>
+            <parameters>$(find one_bot)/config/my_controllers.yaml</parameters>
             <parameters>$(find one_bot)/config/gaz_ros2_ctl_use_sim.yaml</parameters>
         </plugin>
